File: HBW-Sen-PRESS-4_Platine1/HBW-Sen-PRESS-4_Platine1.kicad_pcb (KiCad board)
At the start: 2 copper layers, 86.5 x 33 mm, 40 parts, among them IC1 MC34063AD, IC2 MAX487E, IC3 ATmega328P-A, J1 Nano_Conn, J2 Sensor_Conn, J3 RS485_Conn, J4 24V_Terminal, J5 BUS_Terminal, J6 AVR-ISP-6, Y1 16Mhz

Commit message: Add files via upload
Parts:
- removed R10, R12, R7: 80k, Resistor_SMD:R_0805_2012Metric_Pad1.20x1.40mm_HandSolder
- removed R11, R13, R6, R9: 220k, Resistor_SMD:R_0805_2012Metric_Pad1.20x1.40mm_HandSolder
- J2: footprint Connector_PinHeader_2.54mm:PinHeader_1x12_P2.54mm_Vertical -> TerminalBlock_CUI:TerminalBlock_CUI_TB007-508-06_1x06_P5.08mm_Horizontal
- R1: value 80k -> 100k
- moved R1 39.4 mm to (140.9, 97.0), turned to 0 degrees
- moved J2 27.0 mm to (185.5, 117.9), turned to 90 degrees
Connections:
- IC3 pad 12: /Button -> /D8
- J1 pad 3: /Button -> /A6
- J2 pad 1: /VCC -> /A3
- J2 pad 2: Net-(R1-Pad1) -> /A2
- J2 pad 3: /GND -> /A1
- J2 pad 4: /VCC -> /A0
- J2 pad 5: Net-(J2-Pad5) -> /GND
- J2 pad 6: /GND -> /VCC
- R1 pad 1: Net-(R1-Pad1) -> /VCC
- R1 pad 2: /A0 -> /A6
Routing:
- net /VCC: track 172.5 -> 148.3 mm
- net /A6: track 0.00 -> 18.5 mm, vias 0 -> 2
- net /Button: track 11.8 -> 0.00 mm
- net Net-(J2-Pad11): track 7.43 -> 0.00 mm
- net Net-(R1-Pad1): track 7.42 -> 0.00 mm
- net Net-(J2-Pad5): track 7.42 -> 0.00 mm
- net Net-(R10-Pad1): track 7.41 -> 0.00 mm
- net /A3: track 40.6 -> 44.9 mm
- net /A2: track 38.3 -> 41.5 mm
- net /A1: track 39.4 -> 40.7 mm
- net /A0: track 42.0 -> 42.5 mm
Other:
- board text added: "CC BY-NC-SA 3.0 AT"
- board text added: "V1.1"
- board text removed: "V1.0"
